File: Car_STM/main.brd (EAGLE design)
At the start: 160 x 100 mm, 79 parts, among them IC1 BLUEPILL550, K1 G2RE, K3 TF2-L2-9V, K4 S22, Q1 BC807-40LT1SMD, Q10 BC817-40LT1SMD, Q11 BC817-40LT1SMD, Q12 BC817-40LT1SMD, Q13 BC817-40LT1SMD, Q14 BC817-40LT1SMD, Q15 BC817-40LT1SMD, Q16 BC817-40LT1SMD, Q18 BSS123, Q2 BC807-40LT1SMD, Q3 BSS123, Q4 BSS123, Q5 BC817-40LT1SMD, Q6 BC817-40LT1SMD, Q7 BC817-40LT1SMD, Q8 BSS123, Q9 IRFR5305, X10 1751264, X2 1751248, X3 1751264, X5 1751303, X6 1751264, X7 1751248, X9 1751277

Commit message: V1.2 Two boards from one.
Parts:
- removed IC1: BLUEPILL550, STM32BluePill:DIL40
- removed LM1084: 3V3, linear:TO220H
- added C10, C11, C12, C13, C2, C33, C9: 100nF, eagle-ltspice:C2012
- added C14, C15: 100u, resistor:E2,5-6E
- added C29, C30: 10pF, eagle-ltspice:C2012
- added C31, C32: 6,8pF, eagle-ltspice:C2012
- added D10, D11, D12, D13, D14, D15, D16, D17, D7, D8, D9: (no value), diode:DO-214AC
- added JP1: (no value), pinhead:1X04
- added K10, K11, K2: HY1-12V, relay:HY
- added K12, K13: G2RE, relay:G2RE
- added K14: TF2-L2-9V, relay:TF2
- added K5, K6, K7, K8, K9: S22, Stworzone:LD
- added LM1086: 3V3, v-reg:D2PACK
- added Q17: 8MHz, crystal:HC49UP
- added Q19: MC-306 - 32,768kHz, crystal:MC-306
- added Q20, Q21, Q22, Q23, Q24, Q25, Q26, Q27, Q28, Q29, Q30, Q31: BC817-40LT1SMD, transistor-npn:SOT23-BEC
- added R28, R31, R32, R33, R34, R35, R36, R37, R38, R39, R40, R41: 2k2, resistor:R0805
- added R42, R43: 120, resistor:R0805
- added S1: SWITCH-MOMENTARY-2SMD-4, SparkFun-Electromechanical:TACTILE_SWITCH_TALL
- added SJ1, SJ2, SJ3, SJ4: (no value), jumper:SJ
- added U$2, U$3, U$4, U$5: JACK_3.5, Stworzone:STX3100
- added U$6, U$7: D2_HEAT, Stworzone:D2PACK_HEATSINK
- added U1: STM32F10XRXT6, stm32:TQFP64
- added X11, X13: 1751248, con-phoenix-350:1751248
- added X12, X17, X18: 1751251, con-phoenix-350:1751251
- added X14, X15, X16, X21: (no value), con-ptr500:AK500/2
- added X19, X20, X8: (no value), con-ptr500:AK500/3
- D1, D2: value 1N4004 -> (none); device diode:DO41-10 -> diode:P6-15
- LM317: value 4v2 -> 4V2; device linear:TO220H -> v-reg:D2PACK
- R26, R27: value 240 -> 120
- X1: value (none) -> 1751248; device con-ptr500:AK500/3 -> con-phoenix-350:1751248
- X10: value 1751264 -> (none); device con-phoenix-350:1751264 -> con-ptr500:AK500/2
- moved FUSE2 653.7 mm to (-56.0, 94.0)
- moved FUSE1 650.9 mm to (-56.0, 99.0)
- moved D6 618.8 mm to (-61.9, 78.8)
- moved D4 610.8 mm to (-76.4, 78.8), turned to 180 degrees
- moved R23 607.0 mm to (-67.7, 79.7), turned to 270 degrees
- moved R20 600.5 mm to (-70.6, 79.7), turned to 270 degrees
- moved R30 597.8 mm to (-73.3, 83.5), turned to 180 degrees
- moved Q10 587.8 mm to (-68.4, 85.5)
- moved Q9 587.5 mm to (-66.2, 94.7)
- moved C3 574.0 mm to (33.7, 65.6)
- moved R19 445.2 mm to (-28.0, 95.0), flipped to the bottom, turned to 180 degrees
- moved R18 438.5 mm to (-32.0, 95.0), flipped to the bottom
- moved R17 430.8 mm to (-42.0, 95.0), flipped to the bottom
- moved R10 424.0 mm to (-47.0, 95.0), flipped to the bottom, turned to 180 degrees
- moved R9 393.7 mm to (-57.6, 72.1)
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Connections:
- removed net N$1: 12V_IN.1, D1.A, R18.2
- new net AD_REL1: R33.1, U1.25
- new net AD_REL2: R34.1, U1.37
- new net AD_REL3: R35.1, U1.38
- new net AD_REL4: R36.1, U1.39
- new net AD_REL5: R37.1, U1.40
- new net AD_REL6: R38.1, U1.51
- new net AD_REL7: R39.1, U1.52
- new net BOOT0: SJ2.1, SJ3.1, U1.60
- new net BOOT1: SJ1.1, SJ4.1, U1.28
- new net BT_STER: R28.1, U1.2
- new net CHAR_POW: R31.1, U1.24
- new net C_OSC1: C31.2, Q19.1, U1.3
- new net C_OSC2: C32.2, Q19.4, U1.4
- new net DAY_LIGHT: R32.1, U1.53
- new net LIGHT: U1.8, X12.2
- new net N$100: K14.3, U$5.2
- new net N$101: K14.8, U$5.3
- new net N$50: Q31.B, R41.1
- new net N$52: D7.A, K2.2, Q20.C
- new net N$53: Q20.B, R28.2
- new net N$54: D11.C, K6.COM, X13.1
- new net N$55: Q26.B, R36.2
- new net N$56: D8.A, K5.2, Q21.C
- new net N$57: K2.NO, X11.2
- new net N$58: K2.C@1, K2.C@2, X11.1
- new net N$59: Q21.B, R31.2
- new net N$60: D9.A, K6.2, Q22.C
- new net N$61: Q22.B, R32.2
- new net N$62: D10.A, K7.2, Q23.C
- new net N$63: Q23.B, R33.2
- new net N$64: K5.COM, X8.2
- new net N$65: K7.COM, X14.1
- new net N$66: D14.A, K10.2, Q26.C
- new net N$67: D12.A, K8.2, Q24.C
- new net N$68: Q24.B, R34.2
- new net N$69: K8.COM, X15.1
- new net N$70: Q27.B, R37.2
- new net N$71: D13.A, K9.2, Q25.C
- new net N$72: Q25.B, R35.2
- new net N$73: K9.COM, X16.1
- new net N$74: D15.A, K11.2, Q27.C
- new net N$75: Q28.B, R38.2
- new net N$76: K10.NO, X17.1
- new net N$77: Q29.B, R39.2
- new net N$78: D17.A, K13.2, Q29.C
- new net N$79: K10.NC, X17.3
- new net N$80: D16.A, K12.2
- new net N$81: K10.C@1, K10.C@2, X17.2
- new net N$82: K11.NO, X18.1
- new net N$83: K11.NC, X18.3
- new net N$84: K11.C@1, K11.C@2, X18.2
- new net N$85: K12.S0, K12.S1, X19.1
- new net N$86: K12.O0, K12.O1, X19.3
- new net N$87: K12.P0, K12.P1, X19.2
- new net N$88: K13.S0, K13.S1, X20.1
- new net N$89: K13.O0, K13.O1, X20.3
- new net N$90: K13.P0, K13.P1, X20.2
- new net N$91: K14.2, U$2.2
- new net N$92: K14.9, U$2.3
- new net N$93: K14.7, K3.8
- new net N$94: K14.4, K3.3
- new net N$95: K3.4, U$3.2
- new net N$96: K3.2, U$3.3
- new net N$97: K3.7, U$4.2
- new net N$98: K3.9, U$4.3
- new net N$99: U$2.1, U$3.1, U$4.1, U$5.1
- new net NRST: C33.2, S1.A2, U1.7
- new net OSC_IN: C30.2, Q17.2, U1.5
- new net OSC_OUT: C29.2, Q17.1, U1.6
- new net SWCLK: JP1.3, U1.49
- new net SWDIO: JP1.2, U1.46
- new net V+: 12V_IN.1, D1.A, D10.C, D12.C, D13.C, D8.C, D9.C, K5.1, K5.NO, K6.1, K6.NO, K7.1, K7.NO, K8.1, K8.NO, K9.1, K9.NO, R18.2, X10.1, X10.2
- new net VBAT: C3.+, U1.1
- net +12V: now also D14.C, D15.C, D16.C, D17.C, D7.C, K10.1, K11.1, K12.1, K13.1, K2.1, R42.2, R43.2
- net +3V3: now also C10.2, C11.2, C12.2, C13.2, C2.2, C9.2, JP1.1, LM1086.2, SJ3.2, SJ4.2, U$6.1, U1.13, U1.19, U1.32, U1.48, U1.64, X12.1; no longer C3.+, IC1.1, IC1.18, IC1.40, LM1084.2
- net 12_IN: now also U1.14; no longer IC1.5
- net 12_VOL: now also U1.15; no longer IC1.6
- net AUDIO1: now also R24.2, U1.22; no longer IC1.11
- net AUDIO2: now also R40.1, R41.2, U1.23; no longer IC1.12, R24.2
- net BT_MODE: now also U1.27; no longer IC1.14
- net BT_POW: now also U1.26; no longer IC1.13
- net BT_RX: now also U1.29; no longer IC1.15
- net BT_TX: now also U1.30; no longer IC1.16
- net BUZZER: now also U1.44; no longer IC1.28
- net CAN_POW: now also U1.59; no longer IC1.35
- net CAN_RX: now also U1.61; no longer IC1.36
- net CAN_TX: now also U1.62; no longer IC1.37
- net FUEL_POMP: now also U1.10; no longer IC1.3
- net GND: now also C10.1, C11.1, C12.1, C13.1, C14.-, C15.-, C2.1, C29.1, C30.1, C31.1, C32.1, C33.1, C9.1, D11.A, JP1.4, LM1086.1, Q20.E, Q21.E, Q22.E, Q23.E, Q24.E, Q25.E, Q26.E, Q27.E, Q28.E, Q29.E, Q30.E, Q31.E, S1.B2, SJ1.2, SJ2.2, U1.12, U1.18, U1.31, U1.47, U1.63, X12.3, X13.2, X14.2, X15.2, X16.2, X21.1, X21.2, X8.3; no longer IC1.19, IC1.20, IC1.39, LM1084.1
- net L1: now also U1.16; no longer IC1.7
- net L2: now also U1.17; no longer IC1.8
- net LOCK_CLOSE: now also U1.56; no longer IC1.32
- net LOCK_OPEN: now also U1.57; no longer IC1.33
- net M1: now also U1.20; no longer IC1.9
- net M2: now also U1.21; no longer IC1.10
- net MAIN_POW: now also U1.9; no longer IC1.2
- net MIR_POW: now also U1.11; no longer IC1.4
- net N$22: now also K14.1, R43.1; no longer K3.4, X10.3
- net N$30: now also K14.10, R42.1; no longer K3.2, X10.2
- net N$31: now also K14.5, Q30.C; no longer K3.3, K3.7
- net N$32: now also K14.6, Q31.C; no longer K3.9, X10.1
- net N$33: now also Q30.B, R40.2; no longer K3.8, X10.4
- net N$46: now also C14.+, LM1086.3; no longer LM1084.3
- net N$48: now also X8.1; no longer X1.3
- net N$49: now also C15.+
- net RFID_CS: now also U1.33; no longer IC1.21
- net RFID_INT: now also U1.45; no longer IC1.29
- net RFID_MISO: now also U1.35; no longer IC1.23
- net RFID_MOSI: now also U1.36; no longer IC1.24
- net RFID_POW: now also U1.50; no longer IC1.30
- net RFID_SCK: now also U1.34; no longer IC1.22
- net SIM_POW: now also U1.58; no longer IC1.34
- net SIM_RS: now also U1.41; no longer IC1.25
- net SIM_RX: now also U1.42; no longer IC1.26
- net SIM_TX: now also U1.43; no longer IC1.27
- net VCC: now also U$7.1
- net WATER: now also U1.55; no longer IC1.31
Other:
- board size 160 x 100 mm -> 100 x 100 mm
