File: Car_STM/Power_board.brd (EAGLE design)
At the start: 160 x 100 mm, 31 parts, among them K1 G2RE, K10 HY1-12V, K11 HY1-12V, K12 G2RE, K13 G2RE, K4 S22, K5 S22, K6 S22, K7 S22, K8 S22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

Commit message: V1.22 Logic board in progress
Parts:
- removed 12V_IN, X19, X20: (no value), con-ptr500:AK500/3
- removed JP2: (no value), pinhead:2X09
- removed K12, K13: G2RE, relay:G2RE
- removed X14, X15, X16, X21: (no value), con-ptr500:AK500/2
- removed X17, X18: 1751251, con-phoenix-350:1751251
- added JP1: (no value), pinhead:2X09
- added K2: G2RE, relay:G2RE
- added K3: S22, Stworzone:LD
- added X11, X9: 1751251, con-phoenix-350:1751251
- added X12, X5: (no value), con-ptr500:AK500/3
- added X2, X3, X6, X7: (no value), con-ptr500:AK500/2
- K1: value G2RE -> S22; device relay:G2RE -> Stworzone:LD
- K10, K11: value HY1-12V -> G2RE; device relay:HY -> relay:G2RE
- K8, K9: value S22 -> HY1-12V; device Stworzone:LD -> relay:HY
- X10: device con-ptr500:AK500/2 -> con-ptr500:AK500/3
- X8: device con-ptr500:AK500/3 -> con-ptr500:AK500/2
- moved D3 181.7 mm to (71.0, 91.0), turned to 180 degrees
- moved C2 178.0 mm to (49.0, 76.0)
- moved X13 158.5 mm to (86.1, 84.2), turned to 90 degrees
- moved K4 144.4 mm to (70.3, 56.8), turned to 180 degrees
- moved C1 143.8 mm to (32.0, 77.0)
- moved X8 140.9 mm to (87.5, 35.0), turned to 90 degrees
- moved K7 137.2 mm to (69.7, 83.8), turned to 180 degrees
- moved K9 132.4 mm to (69.4, 18.3)
- moved K1 129.1 mm to (69.7, 74.7), turned to 180 degrees
- moved K6 121.2 mm to (69.7, 39.2), turned to 180 degrees
- moved K8 109.4 mm to (68.9, 26.3)
- moved D2 102.0 mm to (11.5, 69.0), turned to 180 degrees
- moved K5 97.4 mm to (69.1, 48.2), turned to 180 degrees
- moved X4 95.3 mm to (54.7, 10.4)
- moved D1 91.1 mm to (11.9, 80.0), turned to 180 degrees
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Connections:
- net +12V: now also JP1.1, JP1.3, K1.NO, K2.1, K3.1, K5.1, K6.1, K7.1, K8.1, K9.1; no longer JP2.1, JP2.3, K12.1, K13.1, K4.NO
- net AD_REL1: now also JP1.6, K4.2; no longer JP2.6, K7.2
- net AD_REL2: now also JP1.8, K5.2; no longer JP2.8, K8.2
- net AD_REL3: now also JP1.10, K6.2; no longer JP2.10, K9.2
- net AD_REL4: now also JP1.12, K8.2; no longer JP2.12, K10.2
- net AD_REL5: now also JP1.14, K9.2; no longer JP2.14, K11.2
- net AD_REL6: now also JP1.16, K10.2; no longer JP2.16, K12.2
- net AD_REL7: now also JP1.18, K11.2; no longer JP2.18, K13.2
- net AGND: now also JP1.13; no longer JP2.13
- net CHAR_POW: now also JP1.2, K3.2; no longer JP2.2, K5.2
- net DAY_LIGHT: now also JP1.11, K7.2; no longer JP2.11, K6.2
- net FUEL_POMP: now also JP1.9, K2.2; no longer JP2.9, K1.2
- net GND: now also JP1.15, JP1.17, X3.1, X3.2, X5.3, X6.2, X7.2, X8.2; no longer 12V_IN.3, JP2.15, JP2.17, X14.2, X15.2, X16.2, X21.1, X21.2
- net MIR_POW: now also JP1.4, K1.2; no longer JP2.4, K4.2
- net N$18: now also K2.S0, K2.S1; no longer K1.S0, K1.S1
- net N$19: now also K2.P0, K2.P1; no longer K1.P0, K1.P1
- net N$48: now also K1.COM, X5.1; no longer K4.COM, X8.1
- net N$54: now also K7.COM; no longer K6.COM
- net N$64: now also K3.COM, X5.2; no longer K5.COM, X1.2
- net N$65: now also K4.COM, X6.1; no longer K7.COM, X14.1
- net N$69: now also K5.COM, X7.1; no longer K8.COM, X15.1
- net N$73: now also K6.COM, X8.1; no longer K9.COM, X16.1
- net N$76: now also K8.NO, X9.1; no longer K10.NO, X17.1
- net N$79: now also K8.NC, X9.3; no longer K10.NC, X17.3
- net N$81: now also K8.C@1, K8.C@2, X9.2; no longer K10.C@1, K10.C@2, X17.2
- net N$82: now also K9.NO, X11.1; no longer K11.NO, X18.1
- net N$83: now also K9.NC, X11.3; no longer K11.NC, X18.3
- net N$84: now also K9.C@1, K9.C@2, X11.2; no longer K11.C@1, K11.C@2, X18.2
- net N$85: now also K10.S0, K10.S1, X12.1; no longer K12.S0, K12.S1, X19.1
- net N$86: now also K10.O0, K10.O1, X12.3; no longer K12.O0, K12.O1, X19.3
- net N$87: now also K10.P0, K10.P1, X12.2; no longer K12.P0, K12.P1, X19.2
- net N$88: now also K11.S0, K11.S1, X10.1; no longer K13.S0, K13.S1, X20.1
- net N$89: now also K11.O0, K11.O1, X10.3; no longer K13.O0, K13.O1, X20.3
- net N$90: now also K11.P0, K11.P1, X10.2; no longer K13.P0, K13.P1, X20.2
- net V+: now also JP1.5, K3.NO, K4.NO, X1.1, X2.1, X2.2; no longer 12V_IN.1, JP2.5, K5.1, K6.1, K7.1, K8.1, K8.NO, K9.1, K9.NO, X10.1, X10.2
- net V+_2: now also JP1.7, X1.2; no longer 12V_IN.2, JP2.7
Other:
- board size 160 x 100 mm -> 100 x 100 mm
