File: Car_STM/Power_board.brd (EAGLE design)
At the start: 90.2 x 100 mm, 36 parts, among them K1 S22, K10 G2RE, K11 G2RE, K2 G2RE, K3 S22, K4 S22, K5 S22, K6 S22, K7 S22, K8 HY1-12V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

Commit message: V1.25 Just tittle missing
Parts:
- removed JP2: (no value), jumper:JP2
- removed R3: 100k, resistor:R0805
- added Q1: IRFR5305, transistor-power:D-PAK_TO252AA
- added U$1, U$2, U$3, U$4: SCREW_3.2, Stworzone:3,2-PAD
- JP1: device pinhead:2X09 -> pinhead:2X10
- X14: device con-phoenix-254:3POL254 -> con-phoenix-254:2POL254
- moved X15 73.9 mm to (28.0, 32.2), turned to 180 degrees
- moved Q2 63.4 mm to (23.8, 46.0), flipped to the bottom, turned to 270 degrees
- moved JP1 1.25 mm to (7.75, 58.2)
- moved X14 1.00 mm to (28.0, 28.0)
- moved X2 0.10 mm to (36.9, 86.9)
- moved X3 0.10 mm to (26.6, 86.9)
- moved X5 0.10 mm to (81.5, 86.9)
- moved X1 0.10 mm to (12.3, 86.9)
- moved X6 0.10 mm to (48.2, 86.9)
- moved X7 0.10 mm to (58.5, 86.9)
- moved X8 0.10 mm to (68.8, 86.9)
Connections:
- removed net AD_REL7: JP1.18, K11.2
- removed net N$44: JP2.3, Q2.1, R3.1
- removed net N$7: JP2.1, K10.2
- new net FAN: JP1.20, Q1.1
- new net GAS_BUTTON: JP1.14, K9.2
- new net N$6: Q1.4, X14.1
- new net N$9: Q2.4, X15.1
- new net PELTIER: JP1.17, Q2.1
- net +12V: now also Q1.3; no longer R3.2
- net AD_REL1: now also JP1.18, K11.2; no longer JP1.6, K4.2
- net AD_REL2: now also JP1.16, K10.2; no longer JP1.8, K5.2
- net AD_REL3: now also JP1.12, K8.2; no longer JP1.10, K6.2
- net AD_REL4: now also JP1.6, K4.2; no longer JP1.12, K8.2
- net AD_REL5: now also JP1.10, K6.2; no longer JP1.14, K9.2
- net AD_REL6: now also JP1.8, K5.2; no longer JP1.16, JP2.2
- net AGND: now also JP1.19; no longer JP1.17
- net GND: now also U$1.B3,2, U$2.B3,2, U$3.B3,2, U$4.B3,2, X14.2, X15.2
Routing:
- net GAS_BUTTON: track 0.00 -> 108.8 mm, vias 0 -> 2
- net AD_REL7: track 56.4 -> 0.00 mm
- net GND: track 405.8 -> 457.5 mm
- net AD_REL4: track 113.6 -> 74.5 mm, vias 2 -> 0
- net FAN: track 0.00 -> 38.7 mm, vias 0 -> 2
- net AD_REL3: track 84.3 -> 113.6 mm, vias 0 -> 2
- net PELTIER: track 0.00 -> 28.4 mm, vias 0 -> 2
- net N$9: track 0.00 -> 25.1 mm, vias 0 -> 1
- net AD_REL5: track 108.8 -> 84.0 mm, vias 2 -> 0
- net N$6: track 0.00 -> 22.5 mm, vias 0 -> 1
- net AD_REL1: track 76.1 -> 56.4 mm
- net AD_REL6: track 59.6 -> 79.1 mm
- net N$7: track 13.9 -> 0.00 mm
- net +12V: track 293.9 -> 306.7 mm
- net AD_REL2: track 80.1 -> 75.4 mm
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Other:
- board size 90.2 x 100 mm -> 100 x 100 mm
- board text added: "1 - GND 2 - CHAR_POW 3 - MIR_POW"
- board text added: "AD REL 1 NC COM NO"
- board text added: "AD REL 2 NC COM NO"
- board text added: "AD REL 3 NC COM NO"
- board text added: "AD REL 4 12V GND"
- board text added: "AD REL 5 12V GND"
- board text added: "AD REL 6 12V GND"
- board text added: "BEFORE IGNITION"
- board text added: "BIgn AIgn GND"
- board text added: "DAY LIGHT"
- board text added: "FAN"
- board text added: "FUEL_POMP"
- board text added: "GAS BUTTON NC COM NO"
- board text added: "GND"
- board text added: "PELTIER"
- board text added: "POWER IN"
