File: Car_STM/Logic_board.brd (EAGLE design)
At the start: 160 x 100 mm, 151 parts, among them IC1 3V3, IC2 4V2, J1 JACK_3.5, J2 JACK_3.5, J3 JACK_3.5, K1 TF2-L2-9V, K2 TF2-L2-9V, Q1 BC817-40LT1SMD, Q10 BC807-40LT1SMD, Q11 BC817-40LT1SMD, Q12 BC817-40LT1SMD, Q13 BC817-40LT1SMD, Q14 BC807-40LT1SMD, Q15 BC817-40LT1SMD, Q16 BC817-40LT1SMD, Q17 BC817-40LT1SMD, Q18 BC817-40LT1SMD, Q19 BC817-40LT1SMD, Q2 IRFR5305, Q20 BC817-40LT1SMD, Q21 BC817-40LT1SMD, Q22 BC817-40LT1SMD, Q23 BC817-40LT1SMD, Q24 BC817-40LT1SMD, Q25 BC817-40LT1SMD, Q26 BC817-40LT1SMD, Q27 BC817-40LT1SMD, Q28 BC817-40LT1SMD, Q29 BC817-40LT1SMD, Q3 8MHz, Q30 BC817-40LT1SMD, Q31 BC817-40LT1SMD, Q4 MC-306 - 32,768kHz, Q5 BSS84, Q6 BC817-40LT1SMD, Q7 BSS84, Q8 BSS84, Q9 BSS84, U1 STM32F10XRXT6, U2 SIM800L, X1 1751251, X2 1751264, X3 BU-SMA-G, X4 1751264, X5 1751303, X6 1751248, X7 1751248, X8 1751248

Commit message: V1.22 Logic board in progress
Parts:
- removed X1: 1751251, con-phoenix-350:1751251
- removed X2, X4: 1751264, con-phoenix-350:1751264
- removed X5: 1751303, con-phoenix-350:1751303
- removed X8: 1751248, con-phoenix-350:1751248
- added SK1, SK2: (no value), con-hirose-df3:DF3S-04
- added SK3: (no value), con-hirose-df3:DF3S-03
- added SK4, SK6: (no value), con-hirose-df3:DF3S-02
- added SK5: (no value), con-hirose-df3:DF3S-05
- C1, C2, C7, C8: value 100u -> 220uF; device resistor:E2,5-6E -> resistor:PANASONIC_D
- R6, R7, R8: device resistor:0204/7 -> resistor:R0805
- moved C26 489.5 mm to (124.0, 92.8)
- moved R13 480.5 mm to (164.5, 95.0)
- moved SJ5 468.9 mm to (154.2, 93.2)
- moved JP4 426.7 mm to (137.2, 90.0)
- moved Q8 414.0 mm to (179.8, 101.0)
- moved D3 410.2 mm to (167.8, 101.8)
- moved Q9 405.0 mm to (95.5, 46.0), turned to 270 degrees
- moved R47 398.2 mm to (15.0, 53.5), turned to 90 degrees
- moved R46 390.8 mm to (12.5, 53.5), turned to 270 degrees
- moved R45 381.2 mm to (15.0, 49.0), turned to 270 degrees
- moved R44 373.8 mm to (12.5, 49.0), turned to 90 degrees
- moved JP3 353.2 mm to (8.00, 78.0), turned to 270 degrees
- moved JP2 352.4 mm to (7.75, 57.0), turned to 90 degrees
- moved X3 348.9 mm to (93.5, 7.50), turned to 270 degrees
- moved D12 334.3 mm to (52.5, 50.8), turned to 270 degrees
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Connections:
- removed net MIR_POW_P: D4.A, Q21.C
- removed net VBAT: C19.+, U1.1
- net +12V: now also D10.C, D6.C, D7.C, D8.C, D9.C
- net +3V3: now also C19.+, SK2.1, SK3.1, U1.1; no longer X1.1, X4.1
- net AD_REL6_B: now also Q30.C
- net AGND: now also JP2.17; no longer JP2.13
- net CAN_RX: now also SK1.1; no longer X2.1
- net CAN_TX: now also SK1.2; no longer X2.2
- net CHAR_POW_B: now also JP2.15; no longer JP2.2
- net FUEL_POMP: no longer JP2.9
- net FUEL_POMP_B: now also JP2.9
- net GND: now also JP2.2, JP2.4, SK1.4, SK2.4, SK3.3, SK6.1; no longer JP2.15, JP2.17, X1.3, X2.4, X4.4, X5.6
- net LIGHT: now also SK3.2; no longer X1.2
- net M1: now also SK2.2; no longer X4.2
- net M2: now also SK2.3; no longer X4.3
- net MIR_POW_B: now also D4.A, JP2.13, Q21.C; no longer JP2.4
- net N$2: now also SK1.3; no longer X2.3
- net N$20: now also SK4.1; no longer X8.2
- net N$21: now also SK6.2; no longer X5.7, X5.8
- net N$24: now also SK4.2; no longer X8.1
- net RFID_CS: now also SK5.5; no longer X5.1
- net RFID_INT: now also SK5.1; no longer X5.5
- net RFID_MISO: now also SK5.2; no longer X5.4
- net RFID_MOSI: now also SK5.3; no longer X5.3
- net RFID_SCK: now also SK5.4; no longer X5.2
- net V+: now also JP2.7; no longer D10.C, D6.C, D7.C, D8.C, D9.C, JP2.5
- net V+_2: now also JP2.5; no longer JP2.7
Routing:
- net GND: track 0.00 -> 537.2 mm, vias 0 -> 12
- net +3V3: track 0.00 -> 209.3 mm, vias 0 -> 7
- net VCC: track 0.00 -> 120.8 mm, vias 0 -> 3
- net +12V: track 0.00 -> 111.1 mm, vias 0 -> 3
- net L2: track 0.00 -> 88.8 mm, vias 0 -> 2
- net 12_VOL: track 0.00 -> 86.1 mm, vias 0 -> 2
- net 12_IN: track 0.00 -> 84.7 mm, vias 0 -> 2
- net L1: track 0.00 -> 76.2 mm, vias 0 -> 2
- net AD_REL2_B: track 0.00 -> 69.9 mm, vias 0 -> 1
- net AD_REL3_B: track 0.00 -> 65.8 mm, vias 0 -> 1
- net AD_REL4_B: track 0.00 -> 61.9 mm, vias 0 -> 1
- net N$70: track 0.00 -> 59.5 mm, vias 0 -> 1
- net AD_REL5_B: track 0.00 -> 58.4 mm, vias 0 -> 1
- net AD_REL1_B: track 0.00 -> 53.9 mm, vias 0 -> 1
- net N$63: track 0.00 -> 50.5 mm, vias 0 -> 1
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Other:
- board size 160 x 100 mm -> 100 x 100 mm

Commit message: V1.23 First draft of Logic board
Parts:
- moved R13 152.3 mm to (14.8, 67.0), turned to 90 degrees
- moved SJ5 142.8 mm to (14.8, 62.8), turned to 90 degrees
- moved D3 142.8 mm to (32.2, 56.8), flipped to the bottom, turned to 180 degrees
- moved Q8 128.0 mm to (59.5, 57.0)
- moved R12 124.2 mm to (63.3, 56.5), turned to 180 degrees
- moved C14 111.1 mm to (73.2, 53.7), turned to 270 degrees
- moved R24 107.5 mm to (69.8, 62.9), flipped to the bottom
- moved C16 106.0 mm to (87.6, 35.0), turned to 270 degrees
- moved C13 104.9 mm to (75.5, 53.8), turned to 270 degrees
- moved C17 102.4 mm to (89.8, 35.0), turned to 270 degrees
- moved Q16 100.8 mm to (62.8, 67.5)
- moved C18 99.5 mm to (92.1, 35.0), turned to 270 degrees
- moved C15 99.2 mm to (77.8, 53.8), turned to 270 degrees
- moved JP4 97.3 mm to (42.8, 66.8)
- moved R25 87.6 mm to (69.7, 65.4), flipped to the bottom
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Routing:
- net GND: track 537.2 -> 760.8 mm, vias 12 -> 20
- net NRST: track 26.3 -> 176.0 mm, vias 2 -> 4
- net AGND: track 0.00 -> 106.0 mm
- net BT_RX: track 0.00 -> 95.9 mm, vias 0 -> 2
- net BT_TX: track 0.00 -> 93.0 mm, vias 0 -> 2
- net N$18: track 0.00 -> 86.3 mm
- net BT_RES: track 0.00 -> 77.5 mm, vias 0 -> 1
- net +3V3: track 209.3 -> 279.4 mm, vias 7 -> 10
- net RFID_POW: track 0.00 -> 60.6 mm, vias 0 -> 2
- net AUDIO1: track 0.00 -> 46.5 mm, vias 0 -> 2
- net LOCK_OPEN: track 3.01 -> 47.8 mm, vias 0 -> 1
- net BT_A1: track 0.00 -> 42.5 mm, vias 0 -> 1
- net BT_A0: track 0.00 -> 40.9 mm, vias 0 -> 1
- net BT_P1: track 0.00 -> 39.0 mm, vias 0 -> 1
- net BT_POW: track 0.00 -> 38.4 mm, vias 0 -> 2
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Other:
- board size 100 x 100 mm -> 100 x 82.5 mm

Commit message: V1.24 First version of boards ended
Parts:
- added U$1, U$2, U$3, U$4: SCREW_3.2, Stworzone:3,2-PAD
- moved R24 4.37 mm to (70.6, 67.2)
- moved R25 4.10 mm to (70.6, 69.4)
- moved SK3 2.80 mm to (77.7, 4.00)
- moved Q5 1.90 mm to (69.1, 7.25)
- moved SK1 1.90 mm to (67.8, 4.00)
- moved SK4 1.30 mm to (59.0, 4.00)
- moved Q20 0.40 mm to (63.3, 7.63)
- moved J3 0.31 mm to (92.8, 81.9)
- moved R19 0.30 mm to (62.5, 63.9)
- moved R22 0.30 mm to (62.5, 61.4)
- moved X6 0.30 mm to (4.62, 38.0)
Connections:
- net GND: now also U$1.B3,2, U$2.B3,2, U$3.B3,2, U$4.B3,2
Routing:
- net GND: track 760.8 -> 749.2 mm, vias 20 -> 162
- net N$35: track 17.2 -> 12.5 mm, vias 1 -> 2
- net N$22: track 4.33 -> 7.67 mm
- net +12V: track 143.6 -> 141.1 mm
- net +3V3: track 279.4 -> 277.4 mm
- net VCC: track 120.8 -> 122.4 mm
- net N$30: track 4.61 -> 3.07 mm
- net LIGHT: track 28.0 -> 26.9 mm
- net AUDIO1: track 46.5 -> 45.6 mm
- net NRST: track 176.0 -> 175.2 mm
- net N$1: track 3.21 -> 2.41 mm
- net CAN_TX: track 40.6 -> 39.8 mm
- net N$24: track 6.03 -> 6.79 mm
- added copper zone on layer 1, net GND
- added copper zone on layer 16, net GND
Other:
- board text added: "3V3"
- board text added: "A0"
- board text added: "CAN"
- board text added: "CLK"
- board text added: "CS"
- board text added: "DO"
- board text added: "GND"
- board text added: "GSM-ANT"
- board text added: "Light"
- board text added: "Lock"
- board text added: "MI"
- board text added: "MO"
- board text added: "Mirrors"
- board text added: "Motion"
- board text added: "P0"
- board text added: "P10"
- board text added: "P2"
- board text added: "P4"
- board text added: "P6"
- board text added: "P8"
- board text added: "RFID"
- board text added: "SCL"
- board text added: "Water"

Commit message: V1.25 Just tittle missing
Parts:
- added Q32, Q33: BC817-40LT1SMD, transistor-npn:SOT23-BEC
- added R48, R50: 100k, resistor:R0805
- added R49, R51: 2k2, resistor:R0805
- JP2: device pinhead:2X09 -> pinhead:2X10
- moved JP2 1.25 mm to (7.75, 58.2)
Connections:
- net AD_REL5 renamed GAS_BUTTON
- removed net AD_REL6: R42.1, U1.51
- removed net AD_REL7: R43.1, U1.52
- removed net AD_REL7_B: D14.A, JP2.18, Q31.C
- new net FAN: R49.2, U1.38
- new net FAN_B: JP2.20, Q33.C, R48.1
- new net GAS_BUTTON_B: D12.A, JP2.14, Q29.C
- new net N$64: Q33.B, R49.1
- new net N$66: Q32.B, R51.1
- new net PELTIER: R51.2, U1.37
- new net PELTIER_B: JP2.17, Q32.C, R50.1
- net +12V: now also R48.2, R50.2
- net AD_REL1: now also R43.1, U1.52; no longer R37.1, U1.25
- net AD_REL1_B: now also D14.A, JP2.18, Q31.C; no longer D8.A, JP2.6, Q25.C
- net AD_REL2: now also R42.1, U1.51; no longer R38.1, U1.37
- net AD_REL2_B: now also D13.A, JP2.16, Q30.C; no longer D9.A, JP2.8, Q26.C
- net AD_REL3: now also R40.1, U1.39; no longer R39.1, U1.38
- net AD_REL3_B: now also D11.A, JP2.12, Q28.C; no longer D10.A, JP2.10, Q27.C
- net AD_REL4: now also R37.1, U1.25; no longer R40.1, U1.39
- net AD_REL4_B: now also D8.A, JP2.6, Q25.C; no longer D11.A, JP2.12, Q28.C
- net AD_REL5_B: now also D10.A, JP2.10, Q27.C; no longer D12.A, JP2.14, Q29.C
- net AD_REL6_B: now also D9.A, JP2.8, Q26.C; no longer D13.A, JP2.16, Q30.C
- net AGND: now also JP2.19; no longer JP2.17
- net BT_P8: now also R39.1
- net BT_P9: now also R38.1
- net GND: now also Q32.E, Q33.E
Routing:
- net FAN_B: track 0.00 -> 63.3 mm, vias 0 -> 2
- net GAS_BUTTON_B: track 0.00 -> 58.4 mm, vias 0 -> 1
- net BT_P8: track 20.9 -> 73.5 mm, vias 0 -> 2
- net PELTIER_B: track 0.00 -> 47.9 mm, vias 0 -> 2
- net BT_P9: track 27.1 -> 72.5 mm, vias 1 -> 3
- net GND: track 749.2 -> 790.4 mm, vias 162 -> 170
- net AD_REL7_B: track 40.2 -> 0.00 mm
- net FAN: track 0.00 -> 37.7 mm, vias 0 -> 3
- net PELTIER: track 0.00 -> 36.3 mm, vias 0 -> 3
- net AD_REL7: track 31.5 -> 0.00 mm, vias 1 -> 0
- net AD_REL6_B: track 40.4 -> 70.2 mm
- net AD_REL2_B: track 70.2 -> 40.5 mm
- net AD_REL6: track 29.6 -> 0.00 mm, vias 1 -> 0
- net +12V: track 141.1 -> 161.2 mm, vias 4 -> 6
- net AD_REL2: track 13.3 -> 29.6 mm
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