File: Car_STM/Logic_board.sch (EAGLE design)
At the start: 166 parts, among them K1 G2RE, K10 HY1-12V, K11 HY1-12V, K12 G2RE, K13 G2RE, K14 TF2-L2-9V, K2 HY1-12V, K3 TF2-L2-9V, K4 S22, K5 S22, K6 S22, K7 S22, K8 S22, K9 S22, Q1 BC807-40LT1SMD, Q10 BC817-40LT1SMD, Q11 BC817-40LT1SMD, Q12 BC817-40LT1SMD, Q13 BC817-40LT1SMD, Q14 BC817-40LT1SMD, Q15 BC817-40LT1SMD, Q16 BC817-40LT1SMD, Q17 8MHz, Q18 BSS123, Q19 MC-306 - 32,768kHz, Q2 BC807-40LT1SMD, Q20 BC817-40LT1SMD, Q21 BC817-40LT1SMD, Q22 BC817-40LT1SMD, Q23 BC817-40LT1SMD, Q24 BC817-40LT1SMD, Q25 BC817-40LT1SMD, Q26 BC817-40LT1SMD, Q27 BC817-40LT1SMD, Q28 BC817-40LT1SMD, Q29 BC817-40LT1SMD, Q3 BSS123, Q30 BC817-40LT1SMD, Q31 BC817-40LT1SMD, Q4 BSS123, Q5 BC817-40LT1SMD, Q6 BC817-40LT1SMD, Q7 BC817-40LT1SMD, Q8 BSS123, Q9 IRFR5305, U1 STM32F10XRXT6, X1 1751248, X11 1751248, X12 1751251, X13 1751248, X17 1751251, X18 1751251, X2 1751248, X3 1751264, X5 1751303, X6 1751264, X7 1751248, X9 1751277

Commit message: V1.2 Two boards from one.
Parts:
- removed 12V_IN, X19, X20, X8: (no value), con-ptr500:AK500/3
- removed D1, D2: (no value), diode:DIODE-P6-15
- removed D11: (no value), diode:DIODE-DO-214AC
- removed K1, K12, K13: G2RE, relay:G2RE
- removed K10, K11, K2: HY1-12V, relay:HY1-12V
- removed K14, K3: TF2-L2-9V, relay:TF2-L2-9V
- removed K4, K5, K6, K7, K8, K9: S22, Stworzone:S22
- removed R10, R18: 6k8, resistor:R-EU_R0805
- removed R17, R19: 1k8, resistor:R-EU_R0805
- removed U$2, U$3, U$4, U$5: JACK_3.5, Stworzone:JACK_3.5
- removed X10, X14, X15, X16, X21, X4: (no value), con-ptr500:AK500/2
- removed X11, X13: 1751248, con-phoenix-350:1751248
- removed X17, X18: 1751251, con-phoenix-350:1751251
- added JP2: (no value), pinhead:PINHD-1X11
- added JP3: (no value), pinhead:PINHD-1X4
- JP1: device pinhead:PINHD-1X4 -> pinhead:PINHD-1X11
Connections:
- removed net N$100: K141.P, U$5.2
- removed net N$101: K142.P, U$5.5
- removed net N$16: D3.A, K11.2, Q16.C
- removed net N$18: K12.S, K12.S@1, X4-1.KL
- removed net N$19: K12.P, K12.P@1, X4-2.KL
- removed net N$2: 12V_IN-2.KL, D2.A, R10.1
- removed net N$22: K14S.+, R43.1
- removed net N$29: D5.A, K4G$2.2, Q15.C
- removed net N$30: K14R.+, R42.1
- removed net N$34: K3S.+, R27.1
- removed net N$35: K3R.+, R26.1
- removed net N$48: K4G$1.P, X8-1.KL
- removed net N$52: D7.A, K21.2, Q20.C
- removed net N$54: D11.C, K6G$1.P, X13-1.K
- removed net N$56: D8.A, K5G$2.2, Q21.C
- removed net N$57: K22.S, X11-2.K
- removed net N$58: K22.P, K22.P@1, X11-1.K
- removed net N$60: D9.A, K6G$2.2, Q22.C
- removed net N$62: D10.A, K7G$2.2, Q23.C
- removed net N$64: K5G$1.P, X8-2.KL
- removed net N$65: K7G$1.P, X14-1.KL
- removed net N$66: D14.A, K101.2, Q26.C
- removed net N$67: D12.A, K8G$2.2, Q24.C
- removed net N$69: K8G$1.P, X15-1.KL
- removed net N$71: D13.A, K9G$2.2, Q25.C
- removed net N$73: K9G$1.P, X16-1.KL
- removed net N$74: D15.A, K111.2, Q27.C
- removed net N$76: K102.S, X17-1.K
- removed net N$78: D17.A, K131.2, Q29.C
- removed net N$79: K102.O, X17-3.K
- removed net N$80: D16.A, K121.2
- removed net N$81: K102.P, K102.P@1, X17-2.K
- removed net N$82: K112.S, X18-1.K
- removed net N$83: K112.O, X18-3.K
- removed net N$84: K112.P, K112.P@1, X18-2.K
- removed net N$85: K122.S, K122.S@1, X19-1.KL
- removed net N$86: K122.O, K122.O@1, X19-3.KL
- removed net N$87: K122.P, K122.P@1, X19-2.KL
- removed net N$88: K132.S, K132.S@1, X20-1.KL
- removed net N$89: K132.O, K132.O@1, X20-3.KL
- removed net N$90: K132.P, K132.P@1, X20-2.KL
- removed net N$91: K141.O, U$2.2
- removed net N$92: K142.O, U$2.5
- removed net N$93: K142.S, K32.P
- removed net N$94: K141.S, K31.P
- removed net N$95: K31.S, U$3.2
- removed net N$96: K31.O, U$3.5
- removed net N$97: K32.S, U$4.2
- removed net N$98: K32.O, U$4.5
- removed net N$99: U$2.1, U$3.1, U$4.1, U$5.1
- new net A11: JP2.5, R27.2
- new net A12: JP2.6, R26.2
- new net A21: JP2.7, R43.2
- new net A22: JP2.8, R42.2
- new net AD_REL1_B: D10.A, JP1.3, Q23.C
- new net AD_REL2_B: D12.A, JP1.4, Q24.C
- new net AD_REL3_B: D13.A, JP1.5, Q25.C
- new net AD_REL4_B: D14.A, JP1.6, Q26.C
- new net AD_REL5_B: D15.A, JP1.7, Q27.C
- new net AD_REL6_B: D16.A, JP1.8
- new net AD_REL7_B: D17.A, JP1.9, Q29.C
- new net BT_STER_B: D7.A, JP1.10, Q20.C
- new net CHAR_POW_B: D8.A, JP1.1, Q21.C
- new net DAY_LIGHT_B: D9.A, JP1.11, Q22.C
- new net FUEL_POMP_B: D3.A, JP2.9, Q16.C
- new net MIR_POW_B: JP1.2
- new net MIR_POW_P: D5.A, Q15.C
- new net V+_2: JP2.4
- net +12V: now also JP2.1, JP2.2; no longer D1.C, D2.C, K101.1, K11.1, K111.1, K121.1, K131.1, K21.1, K4G$1.S, K4G$2.1, R26.2, R27.2, R42.2, R43.2
- net +3V3: now also JP3.1; no longer JP1.1
- net 12_IN: no longer R10.2, R17.1
- net 12_VOL: no longer R18.1, R19.2
- net GND: now also JP2.10, JP2.11, JP3.4; no longer 12V_IN-3.KL, D11.A, JP1.4, R17.2, R19.1, X13-2.K, X14-2.KL, X15-2.KL, X16-2.KL, X21-1.KL, X21-2.KL, X8-3.KL
- net N$31: now also R43.1; no longer K14S.-
- net N$32: now also R42.1; no longer K14R.-
- net N$36: now also R27.1; no longer K3S.-
- net N$37: now also R26.1; no longer K3R.-
- net SWCLK: now also JP3.3; no longer JP1.3
- net SWDIO: now also JP3.2; no longer JP1.2
- net V+: now also JP2.3; no longer 12V_IN-1.KL, D1.A, K5G$1.S, K5G$2.1, K6G$1.S, K6G$2.1, K7G$1.S, K7G$2.1, K8G$1.S, K8G$2.1, K9G$1.S, K9G$2.1, R18.2, X10-1.KL, X10-2.KL
Other:
- moved on the sheet: C1, C10, C11, C12, C13, C14, C15, C2, C29, C3, C30, C31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

Commit message: V1.21 New BT, audio, big cap on 12V
Parts:
- removed C29, C30: 10pF, eagle-ltspice:CC2012
- removed C31, C32: 6,8pF, eagle-ltspice:CC2012
- removed C33: 100nF, eagle-ltspice:CC2012
- removed D15, D16, D17: (no value), diode:DIODE-DO-214AC
- removed FUSE1: F0.315, resistor:R-EU_R2512
- removed FUSE2: F1.0, resistor:R-EU_R2512
- removed LM1086: 3V3, v-reg:LM317BD2T
- removed LM317: 4V2, v-reg:LM317BD2T
- removed U$1: SIM800L, SIM800L:SIM800L
- removed U$6, U$7: D2_HEAT, Stworzone:D2_HEAT
- removed X12: 1751251, con-phoenix-350:1751251
- removed X9: 1751277, con-phoenix-350:1751277
- added BT1: WT32I, bluegiga_wt32i:WT32I
- added C16, C17, C18, C20, C26: 100nF, eagle-ltspice:CC2012
- added C19: (no value), Cap-Gold:CAP-13,5
- added C21: 2u2, resistor:C-EUC2012
- added C22, C23: 330u/6V3, cap-master:CP-7343
- added C24, C25: 33p, resistor:C-EUC2012
- added D1, D2: LL4148, _hhn_diodes_smd:LL4148
- added D11: (no value), diode:DIODE-DO-214AC
- added H1, H2: D2_HEAT, Stworzone:D2_HEAT
- added IC1: 3V3, v-reg:LM317BD2T
- added IC2: 4V2, v-reg:LM317BD2T
- added J1, J2, J3: JACK_3.5, Stworzone:JACK_3.5
- added JP4: (no value), pinhead:PINHD-1X4
- added K1, K2: TF2-L2-9V, relay:TF2-L2-9V
- added L1, L2: 33n, rcl:L-USL2012C
- added R10, R19: 2k2, resistor:R-EU_R0805
- added R17, R18: 100k, resistor:R-EU_R0805
- added R44, R46: 6k8, resistor:R-EU_R0805
- added R45, R47: 1k8, resistor:R-EU_R0805
- added SJ5: (no value), jumper:SJ
- added U2: SIM800L, SIM800L:SIM800L
- added X4: 1751264, con-phoenix-350:1751264
- added X8: 1751248, con-phoenix-350:1751248
- C10, C9: value 100nF -> 10pF
- C11, C12: value 100nF -> 6,8pF
- C14, C15: value 100u -> 100nF; device resistor:CPOL-EUE2,5-6E -> eagle-ltspice:CC2012
- C2: value 100nF -> 100u; device eagle-ltspice:CC2012 -> resistor:CPOL-EUE2,5-6E
- C3: value (none) -> 100n; device Cap-Gold:CAP-13,5 -> resistor:C-EUC2012
- C7: value 100n -> 100u; device resistor:C-EUC2012 -> resistor:CPOL-EUE2,5-6E
- D3: value (none) -> LL4148; device diode:DIODE-DO-214AC -> _hhn_diodes_smd:LL4148
- D4, D6: value LL4148 -> (none); device _hhn_diodes_smd:LL4148 -> diode:DIODE-DO-214AC
- JP1: device pinhead:PINHD-1X11 -> pinhead:PINHD-1X4
- JP2: device pinhead:PINHD-1X11 -> pinhead:PINHD-2X9
- JP3: device pinhead:PINHD-1X4 -> pinhead:PINHD-2X7
- Q1: value BC807-40LT1SMD -> BC817-40LT1SMD; device transistor-pnp:BC807-40LT1SMD -> transistor-npn:BC817-40LT1SMD
- Q10, Q14: value BC817-40LT1SMD -> BC807-40LT1SMD; device transistor-npn:BC817-40LT1SMD -> transistor-pnp:BC807-40LT1SMD
- Q17: value 8MHz -> BC817-40LT1SMD; device crystal:CRYSTALHC49UP -> transistor-npn:BC817-40LT1SMD
- Q18: value BSS123 -> BC817-40LT1SMD; device transistor-small-signal:BSS123 -> transistor-npn:BC817-40LT1SMD
- Q19: value MC-306 - 32,768kHz -> BC817-40LT1SMD; device crystal:MC-306 -> transistor-npn:BC817-40LT1SMD
- Q2: value BC807-40LT1SMD -> IRFR5305; device transistor-pnp:BC807-40LT1SMD -> transistor-power:IRFR5305
- Q3: value BSS123 -> 8MHz; device transistor-small-signal:BSS123 -> crystal:CRYSTALHC49UP
- Q4: value BSS123 -> MC-306 - 32,768kHz; device transistor-small-signal:BSS123 -> crystal:MC-306
- Q5, Q7: value BC817-40LT1SMD -> BSS84; device transistor-npn:BC817-40LT1SMD -> transistor-small-signal:BSS84
- Q8: value BSS123 -> BSS84; device transistor-small-signal:BSS123 -> transistor-small-signal:BSS84
- Q9: value IRFR5305 -> BSS84; device transistor-power:IRFR5305 -> transistor-small-signal:BSS84
- R1, R2: value 100k -> 2k2
- R11: value 220 -> 100k; device resistor:R-EU_0204/7 -> resistor:R-EU_R0805
- R13: value 2k2 -> 100k
- R14: value 510 -> 1M
- R15: value 240 -> 1M
- R20, R24, R25: value 2k2 -> 120
- R21: value 100 -> 120
- R22: value 100 -> 2k2
- R26, R42, R43: value 120 -> 2k2
- R27: value 120 -> 6k8
- R28: value 2k2 -> 1k8
- R29: value 2k2 -> 6k8
- R3: value 1k8 -> 100k
- R30: value 100k -> 1k8
- R31: value 2k2 -> 510
- R32: value 2k2 -> 240
- R4: value 1k8 -> F0.315; device resistor:R-EU_R0805 -> resistor:R-EU_R2512
- R5: value 6k8 -> F1.0; device resistor:R-EU_R0805 -> resistor:R-EU_R2512
- R6: value 6k8 -> 1k2; device resistor:R-EU_R0805 -> resistor:R-EU_0204/7
- R8: value 1k2 -> 220
- R9: value 2k2 -> 100
- X1: value 1751248 -> 1751251; device con-phoenix-350:1751248 -> con-phoenix-350:1751251
- X2: value 1751248 -> 1751264; device con-phoenix-350:1751248 -> con-phoenix-350:1751264
- X3: value 1751264 -> BU-SMA-G; device con-phoenix-350:1751264 -> con-coax:BU-SMA-G
- X6: value 1751264 -> 1751248; device con-phoenix-350:1751264 -> con-phoenix-350:1751248
Connections:
- removed net A11: JP2.5, R27.2
- removed net A12: JP2.6, R26.2
- removed net A21: JP2.7, R43.2
- removed net A22: JP2.8, R42.2
- removed net BT_MODE: R29.1, U1PORTB_L.PB1
- removed net BT_STER_B: D7.A, JP1.10, Q20.C
- new net AGND: J1.1, J2.1, J3.1, JP2.13
- new net BT_A0: BT1-PIO.AIO0, JP3.1
- new net BT_A1: BT1-PIO.AIO1, JP3.2
- new net BT_LEFT: K12.O, L1.2, R14.2
- new net BT_P0: BT1-PIO.PIO0, JP3.3
- new net BT_P1: BT1-PIO.PIO1, JP3.4
- new net BT_P10: BT1-PIO.PIO10, JP3.13, R13.2
- new net BT_P2: BT1-PIO.PIO2, JP3.5
- new net BT_P3: BT1-PIO.PIO3, JP3.6
- new net BT_P4: BT1-PIO.PIO4, JP3.7
- new net BT_P5: BT1-PIO.PIO5, JP3.8
- new net BT_P6: BT1-PIO.PIO6, JP3.9
- new net BT_P7: BT1-PIO.PIO7, JP3.10
- new net BT_P8: BT1-PIO.PIO8, JP3.11
- new net BT_P9: BT1-PIO.PIO9, JP3.12
- new net BT_RES: D3.A, U1PORTB_L.PB1
- new net BT_RIGHT: K11.O, L2.2, R15.1
- new net N$1: Q5.G, R9.2
- new net N$16: BT1-POWER.RESET, D3.C
- new net N$18: BT1-POWER.VDD_BAT, BT1-POWER.VDD_IO, BT1-POWER.VREG_EN, Q8.D
- new net N$19: BT1-SPI.MOSI, JP4.1
- new net N$2: Q5.D, X2-3.K
- new net N$22: K2S.+, R24.1
- new net N$29: BT1-SPI.MISO, JP4.2
- new net N$30: K2R.+, R25.1
- new net N$34: K1S.+, R20.1
- new net N$35: K1R.+, R21.1
- new net N$48: BT1-AUDIO_OUT.AUDIO_OUT_N_R, C23.+
- new net N$52: C23.-, C25.1, L2.1
- new net N$54: J2.5, K12.S
- new net N$56: J2.2, K11.S
- new net N$57: J1.2, K21.P
- new net N$58: J1.5, K22.P
- new net N$60: U2.NET, X3.1
- new net N$91: J3.2, K21.O
- new net N$92: J3.5, K22.O
- new net N$93: K12.P, K22.S
- new net N$94: K11.P, K21.S
- net +12V: now also D11.C, D12.C, D13.C, D4.C, JP2.3, Q10.E, Q14.E, Q2.S, R20.2, R21.2, R24.2, R25.2, R3.2; no longer D15.C, D16.C, D17.C, D3.C, D7.C, JP2.2, Q1.E, Q2.E, Q9.S, R30.2
- net +3V3: now also C14.2, C15.2, C16.2, C17.2, C18.2, C21.1, C26.2, C5.1, C7.+, H1.K@1, IC1.OUT, JP1.1, Q5.S, Q8.S, Q9.S, R31.2, R32.2, SJ2.2, X1-1.K, X4-1.K; no longer C10.2, C11.2, C12.2, C2.2, C6.1, C8.+, C9.2, JP3.1, LM1086.OUT, R14.2, R15.2, SJ3.2, U$6.K@1, X12-1.K, X3-3.K, X5-7.K, X5-8.K, X6-1.K, X9-3.K
- net 12_IN: now also D1.A, R44.1, R45.2; no longer D4.A
- net 12_VOL: now also R46.1, R47.2
- net 4V2: now also Q7.D, U2.VCC; no longer U$1.VCC
- net AD_REL1: now also R37.1; no longer R33.1
- net AD_REL1_B: now also D8.A, JP2.6, Q25.C; no longer D10.A, JP1.3, Q23.C
- net AD_REL2: now also R38.1; no longer R34.1
- net AD_REL2_B: now also D9.A, JP2.8, Q26.C; no longer D12.A, JP1.4, Q24.C
- net AD_REL3: now also R39.1; no longer R35.1
- net AD_REL3_B: now also D10.A, JP2.10, Q27.C; no longer D13.A, JP1.5, Q25.C
- net AD_REL4: now also R40.1; no longer R36.1
- net AD_REL4_B: now also D11.A, JP2.12, Q28.C; no longer D14.A, JP1.6, Q26.C
- net AD_REL5: now also R41.1; no longer R37.1
- net AD_REL5_B: now also D12.A, JP2.14, Q29.C; no longer D15.A, JP1.7, Q27.C
- net AD_REL6: now also R42.1; no longer R38.1
- net AD_REL6_B: now also D13.A, JP2.16; no longer D16.A, JP1.8
- net AD_REL7: now also R43.1; no longer R39.1
- net AD_REL7_B: now also D14.A, JP2.18, Q31.C; no longer D17.A, JP1.9, Q29.C
- net AUDIO1: now also R19.1, R22.2; no longer R24.2, R25.1
- net AUDIO2: now also R23.1, R26.2; no longer R40.1, R41.2
- net BOOT0: now also SJ1.1; no longer SJ3.1
- net BOOT1: now also SJ3.1; no longer SJ1.1
- net BT_POW: now also R12.1; no longer R22.1
- net BT_RX: now also BT1-UART.RXD; no longer X9-1.K
- net BT_STER: no longer R28.1
- net BT_TX: now also BT1-UART.TXD; no longer X9-2.K
- net BUZZER: now also R8.1; no longer R11.1
- net CAN_POW: now also R9.1; no longer R12.1
- net CAN_RX: now also X2-1.K; no longer X3-1.K
- net CAN_TX: now also X2-2.K; no longer X3-2.K
- net CHAR_POW: now also R35.1; no longer R31.1
- net CHAR_POW_B: now also D6.A, JP2.2, Q23.C; no longer D8.A, JP1.1, Q21.C
- net C_OSC1: now also C11.2, Q4.1; no longer C31.2, Q19.1
- net C_OSC2: now also C12.2, Q4.2; no longer C32.2, Q19.2
- net DAY_LIGHT: now also R36.1; no longer R32.1
- net DAY_LIGHT_B: now also D7.A, JP2.11, Q24.C; no longer D9.A, JP1.11, Q22.C
- net FUEL_POMP: now also JP2.9, R34.1; no longer R13.1
- net FUEL_POMP_B: now also D5.A, Q22.C; no longer D3.A, JP2.9, Q16.C
- net GND: now also BT1-POWER.GND@1, BT1-POWER.GND@2, BT1-POWER.GND@3, BT1-POWER.GND@4, BT1-POWER.GND@5, BT1-POWER.GND@6, BT1-POWER.GND@7, BT1-POWER.GND@8, BT1-UART.!CTS, C14.1, C15.1, C16.1, C17.1, C18.1, C19.-, C2.-, C20.1, C21.2, C24.1, C25.2, C26.1, C3.2, C7.-, IC1.ADJ, JP1.4, JP2.15, JP2.17, Q1.E, Q17.E, Q18.E, Q19.E, R14.1, R15.2, R28.2, R30.2, R45.1, R47.1, R6.1, SJ3.2, U2.GND, X1-3.K, X2-4.K, X3.2, X4-4.K, X5-6.K; no longer C14.-, C15.-, C2.1, C29.1, C3.-, C30.1, C31.1, C32.1, C33.1, C7.2, JP2.10, JP2.11, JP3.4, LM1086.ADJ, Q10.E, Q12.E, Q18.S, Q3.S, Q4.S, Q5.E, Q7.E, Q8.S, R3.2, R4.2, R8.1, SJ2.2, X12-3.K, X6-4.K
- net L1: now also R17.2; no longer R1.2
- net L2: now also R18.1; no longer R2.1
- net LIGHT: now also X1-2.K; no longer X12-2.K
- net LOCK_CLOSE: now also R27.2, R28.1; no longer R4.1, R6.2
- net LOCK_OPEN: now also R29.2, R30.1; no longer R3.1, R5.2
- net M1: now also X4-2.K; no longer X6-2.K
- net M2: now also X4-3.K; no longer X6-3.K
- net MAIN_POW: now also D2.A; no longer D6.A
- net MIR_POW: now also R33.1; no longer R9.1
- net MIR_POW_B: now also JP2.4; no longer JP1.2
- net MIR_POW_P: now also D4.A, Q21.C; no longer D5.A, Q15.C
- net N$10: now also D1.C, R1.2; no longer D4.C, R20.2
- net N$11: now also R8.2; no longer R11.2
- net N$12: now also Q6.C, Q7.G, R11.1; no longer Q3.G, R12.2
- net N$13: now also R12.2; no longer R22.2
- net N$14: now also IC2.ADJ, R6.2; no longer LM317.ADJ, R8.2
- net N$15: now also Q6.B, R10.2; no longer Q3.D, X3-4.K
- net N$17: now also Q22.B, R34.2; no longer Q16.B, R13.2
- net N$20: now also R31.1, X8-2.K; no longer R14.1, X7-2.K
- net N$21: now also Q9.D, X5-7.K, X5-8.K; no longer Q4.D, X5-6.K
- net N$23: now also Q12.B, R17.1; no longer Q14.B, R1.1
- net N$24: now also Q20.B, X8-1.K; no longer Q5.B, X7-1.K
- net N$25: now also R18.2; no longer R2.2
- net N$26: now also Q12.E, Q15.B; no longer Q11.B, Q14.E
- net N$27: now also Q9.G; no longer Q4.G
- net N$28: now also Q21.B, R33.2; no longer Q15.B, R9.2
- net N$3: now also R27.1, X7-1.K; no longer R6.1, X2-1.K
- net N$31: now also K2S.-, Q18.C; no longer Q30.C, R43.1
- net N$32: now also K2R.-, Q19.C; no longer Q31.C, R42.1
- net N$33: now also Q18.B, R23.2; no longer Q30.B, R40.2
- net N$36: now also K1S.-, Q16.C; no longer Q6.C, R27.1
- net N$37: now also K1R.-, Q17.C; no longer Q7.C, R26.1
- net N$38: now also Q16.B, R19.2; no longer Q6.B, R25.2
- net N$39: now also BT1-SPI.SCLK, JP4.3; no longer Q8.D, X9-4.K
- net N$4: now also Q14.C, Q15.C, X6-2.K; no longer Q1.C, Q11.C, X1-2.K
- net N$40: now also Q2.D, R4.1, R5.1; no longer FUSE1.1, FUSE2.1, Q9.D
- net N$41: now also Q17.B, R22.1; no longer Q7.B, R24.1
- net N$42: now also BT1-SPI.!CS, JP4.4; no longer R29.2, X9-5.K
- net N$43: now also Q1.B, R1.1, R2.1; no longer Q10.B, R20.1, R23.1
- net N$44: now also Q1.C, Q2.G, R3.1; no longer Q10.C, Q9.G, R30.1
- net N$45: now also D2.C, R2.2; no longer D6.C, R23.2
- net N$46: now also C1.+, C3.1, IC1.IN, R4.2; no longer C14.+, C7.1, FUSE1.2, LM1086.IN
- net N$47: now also BT1-AUDIO_OUT.AUDIO_OUT_N_L, C22.+; no longer Q18.D, U$1.GND
- net N$49: now also C2.+, IC2.IN, R5.2; no longer C15.+, FUSE2.2, LM317.IN
- net N$5: now also Q10.C, Q11.C, X6-1.K; no longer Q12.C, Q2.C, X1-1.K
- net N$50: now also Q19.B, R26.1; no longer Q31.B, R41.1
- net N$51: now also C22.-, C24.2, L1.1; no longer Q18.G, R21.2
- net N$53: now also R13.1, SJ5.2; no longer Q20.B, R28.2
- net N$55: now also Q28.B, R40.2; no longer Q26.B, R36.2
- net N$59: now also Q23.B, R35.2; no longer Q21.B, R31.2
- net N$6: now also R29.1, X7-2.K; no longer R5.1, X2-2.K
- net N$61: now also Q24.B, R36.2; no longer Q22.B, R32.2
- net N$63: now also Q25.B, R37.2; no longer Q23.B, R33.2
- net N$68: now also Q26.B, R38.2; no longer Q24.B, R34.2
- net N$7: now also Q10.B, Q12.C; no longer Q14.C, Q2.B
- net N$70: now also Q29.B, R41.2; no longer Q27.B, R37.2
- net N$72: now also Q27.B, R39.2; no longer Q25.B, R35.2
- net N$75: now also Q30.B, R42.2; no longer Q28.B, R38.2
- net N$77: now also Q31.B, R43.2; no longer Q29.B, R39.2
- net N$8: now also Q14.B; no longer Q1.B
- net N$9: now also Q11.B; no longer Q12.B
- net NRST: now also C20.2, SJ5.1; no longer C33.2
- net OSC_IN: now also C10.2, Q3.2; no longer C30.2, Q17.2
- net OSC_OUT: now also C9.2, Q3.1; no longer C29.2, Q17.1
- net SIM_POW: now also R10.1; no longer R21.1
- net SIM_RS: now also U2.RST; no longer U$1.RST
- net SIM_RX: now also U2.RXD; no longer U$1.RXD
- net SIM_TX: now also U2.TXD; no longer U$1.TXD
- net SWCLK: now also JP1.3; no longer JP3.3
- net SWDIO: now also JP1.2; no longer JP3.2
- net V+: now also D6.C, D7.C, JP2.5, R46.2; no longer D12.C, D13.C, JP2.3
- net V+_2: now also JP2.7, R44.2; no longer JP2.4
- net VBAT: now also C19.+; no longer C3.+
- net VCC: now also C6.1, C8.+, H2.K@1, IC2.OUT, Q7.S, R11.2; no longer C1.+, C5.1, LM317.OUT, U$7.K@1
- net WATER: now also Q20.C, R32.1; no longer Q5.C, R15.1
Other:
- note removed: "1. zasilanie dżwi niebiesko-zielony między dżwiami a bezp 2. zasilanie okien czerwono-biały między dżwiami a bezp"
- note removed: "lusterka żółto-czerwony i żółto-niebieski, idą z dżwi"
- note removed: "zamek centralny lewo i prawo biało-czarny? pomarańczowo-biały? pomarańczowo-zielony? między centralką a dżwiami"
- note removed: "zasilanie do lusterek niebiesko-zielony między dżwiami a bezp"
- moved on the sheet: C1, C10, C11, C12, C13, C4, C5, C6, C8, C9, D10, D12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

Commit message: V1.22 Logic board in progress
Parts:
- removed X1: 1751251, con-phoenix-350:1751251
- removed X2, X4: 1751264, con-phoenix-350:1751264
- removed X5: 1751303, con-phoenix-350:1751303
- removed X8: 1751248, con-phoenix-350:1751248
- added SK1, SK2: (no value), con-hirose-df3:DF3-04S
- added SK3: (no value), con-hirose-df3:DF3-03S
- added SK4, SK6: (no value), con-hirose-df3:DF3-02S
- added SK5: (no value), con-hirose-df3:DF3-05S
- C1, C2, C7, C8: value 100u -> 220uF; device resistor:CPOL-EUE2,5-6E -> resistor:CPOL-EUD
- R6, R7, R8: device resistor:R-EU_0204/7 -> resistor:R-EU_R0805
Connections:
- removed net MIR_POW_P: D4.A, Q21.C
- removed net VBAT: C19.+, U1AN_POWER.VBAT
- net +12V: now also D10.C, D6.C, D7.C, D8.C, D9.C
- net +3V3: now also C19.+, SK2-1.S, SK3-1.S, U1AN_POWER.VBAT; no longer X1-1.K, X4-1.K
- net AD_REL6_B: now also Q30.C
- net AGND: now also JP2.17; no longer JP2.13
- net CAN_RX: now also SK1-1.S; no longer X2-1.K
- net CAN_TX: now also SK1-2.S; no longer X2-2.K
- net CHAR_POW_B: now also JP2.15; no longer JP2.2
- net FUEL_POMP: no longer JP2.9
- net FUEL_POMP_B: now also JP2.9
- net GND: now also JP2.2, JP2.4, SK1-4.S, SK2-4.S, SK3-3.S, SK6-1.S; no longer JP2.15, JP2.17, X1-3.K, X2-4.K, X4-4.K, X5-6.K
- net LIGHT: now also SK3-2.S; no longer X1-2.K
- net M1: now also SK2-2.S; no longer X4-2.K
- net M2: now also SK2-3.S; no longer X4-3.K
- net MIR_POW_B: now also D4.A, JP2.13, Q21.C; no longer JP2.4
- net N$2: now also SK1-3.S; no longer X2-3.K
- net N$20: now also SK4-1.S; no longer X8-2.K
- net N$21: now also SK6-2.S; no longer X5-7.K, X5-8.K
- net N$24: now also SK4-2.S; no longer X8-1.K
- net RFID_CS: now also SK5-5.S; no longer X5-1.K
- net RFID_INT: now also SK5-1.S; no longer X5-5.K
- net RFID_MISO: now also SK5-2.S; no longer X5-4.K
- net RFID_MOSI: now also SK5-3.S; no longer X5-3.K
- net RFID_SCK: now also SK5-4.S; no longer X5-2.K
- net V+: now also JP2.7; no longer D10.C, D6.C, D7.C, D8.C, D9.C, JP2.5
- net V+_2: now also JP2.5; no longer JP2.7

Commit message: V1.24 First version of boards ended
Parts:
- added U$1, U$2, U$3, U$4: SCREW_3.2, Stworzone:SCREW_3.2
Connections:
- net GND: now also U$1.MOUNT, U$2.MOUNT, U$3.MOUNT, U$4.MOUNT
Changed lines of the file:
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@@
 <part name="SK6" library="con-hirose-df3" deviceset="DF3-02S" device=""/>
 <part name="SK5" library="con-hirose-df3" deviceset="DF3-05S" device=""/>
+<part name="GND46" library="supply1" deviceset="GND" device=""/>
+<part name="U$1" library="Stworzone" deviceset="SCREW_3.2" device=""/>
+<part name="U$2" library="Stworzone" deviceset="SCREW_3.2" device=""/>
+<part name="U$3" library="Stworzone" deviceset="SCREW_3.2" device=""/>
+<part name="U$4" library="Stworzone" deviceset="SCREW_3.2" device=""/>
 </parts>
 <sheets>
@@
 <instance part="SK5" gate="-4" x="-104.14" y="-15.24"/>
 <instance part="SK5" gate="-5" x="-104.14" y="-7.62"/>
+<instance part="GND46" gate="1" x="-175.26" y="-121.92"/>
+<instance part="U$1" gate="G$1" x="-190.5" y="-111.76" rot="R90"/>
+<instance part="U$2" gate="G$1" x="-180.34" y="-111.76" rot="R90"/>
+<instance part="U$3" gate="G$1" x="-170.18" y="-111.76" rot="R90"/>
+<instance part="U$4" gate="G$1" x="-160.02" y="-111.76" rot="R90"/>
 </instances>
 <busses>
@@
 <pinref part="GND16" gate="1" pin="GND"/>
 </segment>
+<segment>
+<wire x1="-190.5" y1="-114.3" x2="-190.5" y2="-116.84" width="0.1524" layer="91"/>
+<wire x1="-190.5" y1="-116.84" x2="-180.34" y2="-116.84" width="0.1524" layer="91"/>
+<wire x1="-180.34" y1="-114.3" x2="-180.34" y2="-116.84" width="0.1524" layer="91"/>
+<pinref part="U$1" gate="G$1" pin="MOUNT"/>
+<pinref part="U$2" gate="G$1" pin="MOUNT"/>
+<pinref part="U$3" gate="G$1" pin="MOUNT"/>
+<wire x1="-180.34" y1="-116.84" x2="-175.26" y2="-116.84" width="0.1524" layer="91"/>
+<wire x1="-175.26" y1="-116.84" x2="-170.18" y2="-116.84" width="0.1524" layer="91"/>
+<wire x1="-170.18" y1="-116.84" x2="-170.18" y2="-114.3" width="0.1524" layer="91"/>
+<pinref part="U$4" gate="G$1" pin="MOUNT"/>
+<wire x1="-170.18" y1="-116.84" x2="-160.02" y2="-116.84" width="0.1524" layer="91"/>
+<wire x1="-160.02" y1="-116.84" x2="-160.02" y2="-114.3" width="0.1524" layer="91"/>
+<pinref part="GND46" gate="1" pin="GND"/>
+<wire x1="-175.26" y1="-119.38" x2="-175.26" y2="-116.84" width="0.1524" layer="91"/>
+</segment>
 </net>

Commit message: V1.25 Just tittle missing
Parts:
- added Q32, Q33: BC817-40LT1SMD, transistor-npn:BC817-40LT1SMD
- added R48, R50: 100k, resistor:R-EU_R0805
- added R49, R51: 2k2, resistor:R-EU_R0805
- JP2: device pinhead:PINHD-2X9 -> pinhead:PINHD-2X10
Connections:
- net AD_REL5 renamed GAS_BUTTON
- removed net AD_REL6: R42.1, U1PORTC_H.PC10
- removed net AD_REL7: R43.1, U1PORTC_H.PC11
- removed net AD_REL7_B: D14.A, JP2.18, Q31.C
- new net FAN: R49.2, U1PORTC_L.PC7
- new net FAN_B: JP2.20, Q33.C, R48.1
- new net GAS_BUTTON_B: D12.A, JP2.14, Q29.C
- new net N$64: Q33.B, R49.1
- new net N$66: Q32.B, R51.1
- new net PELTIER: R51.2, U1PORTC_L.PC6
- new net PELTIER_B: JP2.17, Q32.C, R50.1
- net +12V: now also R48.2, R50.2
- net AD_REL1: now also R43.1, U1PORTC_H.PC11; no longer R37.1, U1PORTC_L.PC5
- net AD_REL1_B: now also D14.A, JP2.18, Q31.C; no longer D8.A, JP2.6, Q25.C
- net AD_REL2: now also R42.1, U1PORTC_H.PC10; no longer R38.1, U1PORTC_L.PC6
- net AD_REL2_B: now also D13.A, JP2.16, Q30.C; no longer D9.A, JP2.8, Q26.C
- net AD_REL3: now also R40.1, U1PORTC_H.PC8; no longer R39.1, U1PORTC_L.PC7
- net AD_REL3_B: now also D11.A, JP2.12, Q28.C; no longer D10.A, JP2.10, Q27.C
- net AD_REL4: now also R37.1, U1PORTC_L.PC5; no longer R40.1, U1PORTC_H.PC8
- net AD_REL4_B: now also D8.A, JP2.6, Q25.C; no longer D11.A, JP2.12, Q28.C
- net AD_REL5_B: now also D10.A, JP2.10, Q27.C; no longer D12.A, JP2.14, Q29.C
- net AD_REL6_B: now also D9.A, JP2.8, Q26.C; no longer D13.A, JP2.16, Q30.C
- net AGND: now also JP2.19; no longer JP2.17
- net BT_P8: now also R39.1
- net BT_P9: now also R38.1
- net GND: now also Q32.E, Q33.E
Other:
- moved on the sheet: D10, D11, D12, D13, D14, D8, D9, Q25, Q26, Q27, Q28, Q29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
